File: Sensado_Control_DC_5/Sensado_Control_DC_5.kicad_pcb (KiCad board)
At the start: 2 copper layers, 100 x 100 mm, 92 parts, among them J1 Jumper, J2 Jumper, J3 Jumper, P1 R_FUENTE_CON, P10 GPIO, P11 CONM_R1, P2 I_+, P3 I_-, P4 POWER, P5 RS-232, P6 I2C, P7 SPI, P8 GND_REG, P9 RESET, Q1 NMOS, Q10 PMOS, Q11 NMOS, Q12 NMOS, Q13 NMOS, Q14 PMOS, Q15 PMOS, Q16 PMOS, Q2 NMOS, Q3 NMOS, Q4 NMOS, Q5 NMOS, Q6 PMOS, Q7 PMOS, Q8 PMOS, Q9 PMOS, U1 Atmega328PA, U2 ACS_712, U3 LD1117S50TR_FINAL

Commit message: Version avanzada PCB
Parts:
- removed P11: CONM_R1, Socket_Strips:Socket_Strip_Straight_1x02_Pitch2.54mm
- C4: value 1nF -> 1nF_THT; footprint Capacitors_SMD:C_1206_HandSoldering -> Capacitors_THT:C_Disc_D5.0mm_W2.5mm_P2.50mm
- R6: footprint Resistors_THT:R_Axial_DIN0207_L6.3mm_D2.5mm_P10.16mm_Horizontal -> Resistors_THT:R_Axial_DIN0207_L6.3mm_D2.5mm_P7.62mm_Horizontal
- moved C9 173.7 mm to (87.2, 81.1)
- moved R45 169.3 mm to (101.2, 67.0), turned to 90 degrees
- moved J3 167.2 mm to (92.4, 87.3), turned to 180 degrees
- moved C6 160.1 mm to (101.2, 73.2), turned to 270 degrees
- moved R46 156.7 mm to (97.2, 81.1)
- moved C4 154.2 mm to (108.7, 124.5)
- moved R43 147.1 mm to (100.3, 125.5)
- moved U2 140.5 mm to (105.9, 131.6), turned to 90 degrees
- moved C5 138.7 mm to (104.0, 124.3), turned to 270 degrees
- moved P3 137.0 mm to (110.4, 142.9)
- moved C7 129.9 mm to (132.2, 135.5)
- moved U3 128.4 mm to (92.4, 71.3), turned to 90 degrees
- moved D2 119.9 mm to (101.3, 62.5), turned to 270 degrees
- moved P8 110.6 mm to (88.8, 87.3)
- moved C8 108.3 mm to (132.3, 139.9)
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Connections:
- C5 pad 2: Net-(C5-Pad2) -> /5V
- P4 pad 1: /V_FUENTE -> /GND
- P4 pad 2: /GND -> /V_FUENTE
- R1 pad 1: /VCONTROL_1 -> /VCONTROL_5
- R2 pad 1: /VCONTROL_2 -> /VCONTROL_4
- R27 pad 1: /VCONTROL_6 -> /VCONTROL_7
- R28 pad 1: /VCONTROL_7 -> /VCONTROL_2
- R29 pad 1: /VCONTROL_8 -> /VCONTROL_1
- R4 pad 1: /VCONTROL_4 -> /VCONTROL_6
- R43 pad 2: Net-(C5-Pad2) -> /5V
- R5 pad 1: /VCONTROL_5 -> /VCONTROL_8
- U2 pad 8: Net-(C5-Pad2) -> /5V
Routing:
- net /VOUT: track 21.1 -> 494.1 mm, vias 0 -> 19
- net /5V: track 20.5 -> 201.7 mm, vias 3 -> 7
- net /VFB: track 0.00 -> 158.0 mm
- net /VCONTROL_8: track 3.84 -> 115.2 mm, vias 1 -> 4
- net /VCONTROL_7: track 3.83 -> 98.5 mm, vias 1 -> 4
- net /VCONTROL_5: track 5.04 -> 88.6 mm, vias 1 -> 2
- net /VCONTROL_2: track 2.05 -> 84.4 mm, vias 1 -> 4
- net /VOUT_SENS: track 0.00 -> 60.6 mm
- net /VCONTROL_4: track 3.91 -> 63.9 mm, vias 1 -> 2
- net /VCONTROL_1: track 2.05 -> 58.2 mm, vias 1 -> 2
- net /GND: track 29.3 -> 77.2 mm, vias 10 -> 21
- net /VCONTROL_3: track 2.74 -> 45.0 mm, vias 1 -> 2
- net /VCONTROL_6: track 2.76 -> 34.1 mm, vias 1 -> 2
- net /V_FUENTE: track 0.00 -> 31.1 mm
- net /I_SENS-: track 0.00 -> 22.0 mm
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- added copper zone on B.Cu, net /GND
