File: Sensado_Control_DC_5/_autosave-Sensado_Control_DC_5.kicad_pcb (KiCad board)
At the start: 2 copper layers, 100 x 100 mm, 91 parts, among them J1 Jumper, J2 Jumper, J3 Jumper, P1 R_FUENTE_CON, P10 GPIO, P2 I_+, P3 I_-, P4 POWER, P5 RS-232, P6 I2C, P7 SPI, P8 GND_REG, P9 RESET, Q1 NMOS, Q10 PMOS, Q11 NMOS, Q12 NMOS, Q13 NMOS, Q14 PMOS, Q15 PMOS, Q16 PMOS, Q2 NMOS, Q3 NMOS, Q4 NMOS, Q5 NMOS, Q6 PMOS, Q7 PMOS, Q8 PMOS, Q9 PMOS, U1 Atmega328PA, U2 ACS_712, U3 LD1117S50TR_FINAL

Commit message: Isletas y clock añadido a la PCB
Parts:
- added Y1: XRCHA_16M, Huellas:Crystal_SMD_XRCHA_Murata_Serie_W2,5mm_L2,0mm, F.Cu at (140.1, 138.6)
- C7, C8: value 18pF -> 8pF
- U1: footprint Housings_QFP:LQFP-32_7x7mm_Pitch0.8mm -> Housings_QFP:TQFP-32_7x7mm_Pitch0.8mm
- moved C7 10.4 mm to (142.6, 136.3), turned to 90 degrees
- moved C8 10.3 mm to (142.6, 141.0), turned to 270 degrees
Routing:
- net /CLK1: track 5.59 -> 13.3 mm
- net /CLK2: track 5.75 -> 13.4 mm
- net /GND: track 77.2 -> 80.4 mm, vias 21 -> 23
- added copper zone on F.Cu, net (none)
- added copper zone on F.Cu, net /5V
- added copper zone on F.Cu, net /GND
- added copper zone on F.Cu, net /V_FUENTE
